File: Elec/Broche lumineuse/Broche lumineuse.sch (KiCad schematic (older format))
At the start: 30 parts, among them J1 USB_B_Micro, J2 Conn_01x02, J3 Conn_01x02, J4 Conn_01x03, J5 Conn_01x06_Male, Q1 PMV20XNEAR, Q2 DMN2215UDM-7, U1 ATtiny85V-10MU, U2 MMA8453Q, U3 MCP1700-2502E_SOT23, U4 MCP73831-2-OT, U6 SN74LVC1T45DBV, U7 BQ29707DSER

Commit message: Maj schéma suivant tests sur rev.1; Maj temporaire du PCB
Parts:
- removed U6: SN74LVC1T45DBV, Package_TO_SOT_SMD:SOT-23-6, symbol Broche-lumineuse-rescue:SN74LVC1T45DBV-Logic_LevelTranslator
- added R9: 56kR, Resistor_SMD:R_0402_1005Metric, symbol Device:R
- added U6: SN74LV1T34DBVR, Package_TO_SOT_SMD:SOT-353_SC-70-5, symbol SN74LV1T34:SN74LV1T34DBVR
- C1, C2, C3, C4, C5, C6, C7, C8: symbol Broche-lumineuse-rescue:C-Device -> Device:C
- D1: symbol Broche-lumineuse-rescue:LED-Device -> Device:LED
- J1: symbol Broche-lumineuse-rescue:USB_B_Micro-Connector -> Connector:USB_B_Micro
- J2, J3: symbol Broche-lumineuse-rescue:Conn_01x02-Connector_Generic -> Connector_Generic:Conn_01x02
- J4: symbol Broche-lumineuse-rescue:Conn_01x03-Connector_Generic -> Connector_Generic:Conn_01x03
- J5: symbol Broche-lumineuse-rescue:Conn_01x06_Male-Connector -> Connector:Conn_01x06_Male
- Q1: symbol Broche-lumineuse-rescue:BSS138-Transistor_FET -> Transistor_FET:BSS138
- Q2: symbol Broche-lumineuse-rescue:DMN2215UDM-7-eec -> DMN2215UDM-7:DMN2215UDM-7
- R1, R2, R3, R4, R5, R6, R7, R8: symbol Broche-lumineuse-rescue:R-Device -> Device:R
- U1: symbol Broche-lumineuse-rescue:ATtiny85V-10MU-MCU_Microchip_ATtiny -> MCU_Microchip_ATtiny:ATtiny85V-10MU
- U3: symbol Broche-lumineuse-rescue:MCP1700-2502E_SOT23-Regulator_Linear -> Regulator_Linear:MCP1700-2502E_SOT23
- U4: symbol Broche-lumineuse-rescue:MCP73831-2-OT-Battery_Management -> Battery_Management:MCP73831-2-OT
- U7: symbol Broche-lumineuse-rescue:BQ297xy-Battery_Management -> Battery_Management:BQ297xy
Connections:
- net MISO is gone; now on net SCL: J5.2 (Pin_2), U1.12 (PB1)
- net +2V5: now also U2.7 (SA0)
- net +BATT: now also U6.5 (VCC)
- net GND: now also R9.2; no longer J1.6 (Shield)
- net LED_CMD: now also U6.2 (A)
- net LED_INPUT: now also U6.4 (Y)
- net LED_PWR: now also R9.1
- net SCL: no longer J5.3 (Pin_3), U1.14 (PB2)
- net INT0: now reaches U2.9 (INT2)
- net INT0: now also J5.3 (Pin_3), U1.14 (PB2)
- net LED_GND: now reaches J4.3 (Pin_3), Q1.3 (D)
- net LED_GND: now also U6.3 (GND)
Other:
- moved on the sheet: C3, C6, Q1
